File: eagle/ScarfSwarm/schematic.brd (EAGLE design)
At the start: 21.6 x 50.8 mm, 5 parts

Commit message: rearrange JST connection for strip, bump version
Connections:
- net N$13: now also SCARFYMCSCARFFACE.22; no longer SCARFYMCSCARFFACE.23
- net N$8: now also SCARFYMCSCARFFACE.23; no longer SCARFYMCSCARFFACE.22
Routing:
- net N$13: track 8.26 -> 9.75 mm
- net N$8: track 13.3 -> 14.7 mm
Other:
- board text added: "v1.3.0 Aug 2, 2019"
- board text removed: "v1.2.0 Aug 2, 2019"
Changed lines of the file:
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@@
 <drawing>
 <settings>
-<setting alwaysvectorfont="no"/>
+<setting alwaysvectorfont="yes"/>
 <setting verticaltext="up"/>
 </settings>
 <grid distance="50" unitdist="mil" unit="mil" style="lines" multiple="1" display="yes" altdistance="5" altunitdist="mil" altunit="mil"/>
 <layers>
-<layer number="1" name="Top" color="4" fill="1" visible="no" active="yes"/>
+<layer number="1" name="Top" color="4" fill="1" visible="yes" active="yes"/>
 <layer number="16" name="Bottom" color="1" fill="1" visible="no" active="yes"/>
-<layer number="17" name="Pads" color="2" fill="1" visible="no" active="yes"/>
-<layer number="18" name="Vias" color="2" fill="1" visible="no" active="yes"/>
-<layer number="19" name="Unrouted" color="6" fill="1" visible="no" active="yes"/>
-<layer number="20" name="Dimension" color="24" fill="1" visible="no" active="yes"/>
-<layer number="21" name="tPlace" color="7" fill="1" visible="no" active="yes"/>
-<layer number="22" name="bPlace" color="7" fill="1" visible="yes" active="yes"/>
-<layer number="23" name="tOrigins" color="15" fill="1" visible="no" active="yes"/>
+<layer number="17" name="Pads" color="2" fill="1" visible="yes" active="yes"/>
+<layer number="18" name="Vias" color="2" fill="1" visible="yes" active="yes"/>
+<layer number="19" name="Unrouted" color="6" fill="1" visible="yes" active="yes"/>
+<layer number="20" name="Dimension" color="24" fill="1" visible="yes" active="yes"/>
+<layer number="21" name="tPlace" color="7" fill="1" visible="yes" active="yes"/>
+<layer number="22" name="bPlace" color="7" fill="1" visible="no" active="yes"/>
+<layer number="23" name="tOrigins" color="15" fill="1" visible="yes" active="yes"/>
 <layer number="24" name="bOrigins" color="15" fill="1" visible="no" active="yes"/>
-<layer number="25" name="tNames" color="7" fill="1" visible="no" active="yes"/>
+<layer number="25" name="tNames" color="7" fill="1" visible="yes" active="yes"/>
 <layer number="26" name="bNames" color="7" fill="1" visible="no" active="yes"/>
 <layer number="27" name="tValues" color="7" fill="1" visible="no" active="yes"/>
@@
 <layer number="37" name="tTest" color="7" fill="1" visible="no" active="yes"/>
 <layer number="38" name="bTest" color="7" fill="1" visible="no" active="yes"/>
-<layer number="39" name="tKeepout" color="4" fill="11" visible="no" active="yes"/>
+<layer number="39" name="tKeepout" color="4" fill="11" visible="yes" active="yes"/>
 <layer number="40" name="bKeepout" color="1" fill="11" visible="no" active="yes"/>
-<layer number="41" name="tRestrict" color="4" fill="10" visible="no" active="yes"/>
+<layer number="41" name="tRestrict" color="4" fill="10" visible="yes" active="yes"/>
 <layer number="42" name="bRestrict" color="1" fill="10" visible="no" active="yes"/>
 <layer number="43" name="vRestrict" color="2" fill="10" visible="no" active="yes"/>
@@
 <layer number="49" name="Reference" color="7" fill="1" visible="no" active="yes"/>
 <layer number="50" name="dxf" color="7" fill="1" visible="no" active="no"/>
-<layer number="51" name="tDocu" color="7" fill="1" visible="no" active="yes"/>
+<layer number="51" name="tDocu" color="7" fill="1" visible="yes" active="yes"/>
 <layer number="52" name="bDocu" color="7" fill="1" visible="no" active="yes"/>
 <layer number="53" name="tGND_GNDA" color="7" fill="9" visible="no" active="no"/>
@@
 <text x="12.446" y="44.323" size="0.8128" layer="22" rot="SMR270">11/MO</text>
 <text x="17.526" y="44.323" size="0.8128" layer="22" rot="SMR270">12/MI</text>
-<text x="15.367" y="-0.381" size="0.8128" layer="22" rot="MR0">v1.2.0 Aug 2, 2019</text>
+<text x="14.097" y="-0.381" size="0.8128" layer="22" rot="MR0">v1.3.0 Aug 2, 2019</text>
 <text x="13.97" y="38.1" size="1.016" layer="22" rot="MR0">Party on Garth.</text>
 <text x="13.97" y="12.7" size="1.016" layer="22" rot="MR0">Party on Wayne.</text>
@@
 <signal name="N$8">
 <contactref element="LEDSTRIP" pad="2"/>
-<contactref element="SCARFYMCSCARFFACE" pad="22"/>
-<wire x1="10.795" y1="24.765" x2="1.905" y2="24.765" width="0.1524" layer="16"/>
-<wire x1="10.795" y1="20.828" x2="10.795" y2="24.765" width="0.1524" layer="16"/>
-<wire x1="1.905" y1="24.765" x2="1.905" y2="25.273" width="0.1524" layer="16"/>
+<contactref element="SCARFYMCSCARFFACE" pad="23"/>
+<wire x1="10.795" y1="20.828" x2="10.795" y2="18.415" width="0.1524" layer="16"/>
+<wire x1="10.795" y1="18.415" x2="10.16" y2="17.78" width="0.1524" layer="16"/>
+<wire x1="10.16" y1="17.78" x2="5.08" y2="17.78" width="0.1524" layer="16"/>
+<wire x1="5.08" y1="17.78" x2="3.81" y2="19.05" width="0.1524" layer="16"/>
+<wire x1="3.81" y1="20.828" x2="1.905" y2="22.733" width="0.1524" layer="16"/>
+<wire x1="3.81" y1="19.05" x2="3.81" y2="20.828" width="0.1524" layer="16"/>
 </signal>
 <signal name="N$9">
@@
 <wire x1="5.715" y1="14.605" x2="5.715" y2="20.828" width="1.27" layer="1"/>
 <wire x1="8.128" y1="12.192" x2="5.715" y2="14.605" width="1.27" layer="1"/>
-<wire x1="18.415" y1="38.735" x2="17.145" y2="40.005" width="0.1524" layer="16"/>
-<wire x1="18.415" y1="6.985" x2="18.415" y2="38.735" width="0.1524" layer="16"/>
-<wire x1="17.78" y1="6.35" x2="18.415" y2="6.985" width="0.1524" layer="16"/>
-<wire x1="8.255" y1="6.35" x2="17.78" y2="6.35" width="0.1524" layer="16"/>
-<wire x1="8.255" y1="3.175" x2="8.255" y2="6.35" width="0.1524" layer="16"/>
-<wire x1="17.145" y1="40.005" x2="17.145" y2="40.513" width="0.1524" layer="16"/>
-<wire x1="8.255" y1="3.175" x2="8.128" y2="3.048" width="0.1524" layer="16"/>
+<wire x1="18.415" y1="38.735" x2="17.145" y2="40.005" width="0.254" layer="16"/>
+<wire x1="18.415" y1="6.985" x2="18.415" y2="38.735" width="0.254" layer="16"/>
+<wire x1="17.78" y1="6.35" x2="18.415" y2="6.985" width="0.254" layer="16"/>
+<wire x1="8.255" y1="6.35" x2="17.78" y2="6.35" width="0.254" layer="16"/>
+<wire x1="8.255" y1="3.175" x2="8.255" y2="6.35" width="0.254" layer="16"/>
+<wire x1="17.145" y1="40.005" x2="17.145" y2="40.513" width="0.254" layer="16"/>
+<wire x1="8.255" y1="3.175" x2="8.128" y2="3.048" width="0.254" layer="16"/>
 </signal>
 <signal name="N$13">
 <contactref element="LEDSTRIP" pad="3"/>
-<contactref element="SCARFYMCSCARFFACE" pad="23"/>
-<wire x1="8.255" y1="22.225" x2="1.905" y2="22.225" width="0.1524" layer="16"/>
-<wire x1="8.255" y1="20.828" x2="8.255" y2="22.225" width="0.1524" layer="16"/>
-<wire x1="1.905" y1="22.225" x2="1.905" y2="22.733" width="0.1524" layer="16"/>
+<contactref element="SCARFYMCSCARFFACE" pad="22"/>
+<wire x1="8.255" y1="20.828" x2="8.255" y2="23.495" width="0.1524" layer="16"/>
+<wire x1="6.477" y1="25.273" x2="1.905" y2="25.273" width="0.1524" layer="16"/>
+<wire x1="8.255" y1="23.495" x2="6.477" y2="25.273" width="0.1524" layer="16"/>
 </signal>
 <signal name="5V">
